File: Eagle Files - LED module electronic board/Schematic.sch (EAGLE design)
At the start: 14 parts, among them IC1 AMS1117-1.5, IC2 LM358N, J1 2.54 CONN, J2 2.54 CONN, Q1 P16NF06L

Commit message: Update
Parts:
- removed J1, J2: 2.54 CONN, SparkFun-Connectors:CONN_02
- removed Q1: P16NF06L, adafruit:MOSFET-NGDS_TO220V
- removed R3: 10k, LED-microscope-library:POTENTIOMETER_3-PIN
- added Q2: P16NF06L, transistor-power:PMOSFET_NTO220BV
- added U$1: (no value), untitled:POT-SWITCH
- added U$3, U$4: (no value), untitled:SCREW-TERM
Connections:
- new net N$10: IC2B.+IN, U$1G$1.P$2
- net GND: now also U$1G$1.P$3, U$3.1; no longer J1.1, R3.1
- net N$1: now also U$1G$2.P$2, U$3.2; no longer IC2B.+IN, R3.3
- net N$4: now also U$1G$1.P$1; no longer R3.2
- net N$5: now also Q2.D, U$4.2; no longer J2.2, Q1.D
- net N$7: now also Q2.G; no longer Q1.G
- net N$9: now also Q2.S; no longer Q1.S
- net VCC: now also U$1G$2.P$1, U$4.1; no longer J1.2, J2.1
Other:
- moved on the sheet: C3, IC2B, R4, R5, R6

Commit message: Major changes!
Major changes! Do not use older version, pins swapped in V-regulator.
Parts:
- removed IC1: AMS1117-1.5, linear:LM340MP-05
- added U$2: VREG-AMS1117-1.5, untitled:VREG-AMS1117-1.5
Connections:
- net GND: now also U$2.GND; no longer IC1.GND
- net N$3: now also U$2.OUT, U$2.OUT@1; no longer IC1.VO
- net VCC: now also U$2.IN; no longer IC1.VI
Changed lines of the file:
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@@
 </classes>
 <parts>
-<part name="IC1" library="linear" library_urn="urn:adsk.eagle:library:262" deviceset="LM340?-*" device="MP" package3d_urn="urn:adsk.eagle:package:28541/2" technology="05" value="AMS1117-1.5"/>
 <part name="GND1" library="supply1" library_urn="urn:adsk.eagle:library:371" deviceset="GND" device="">
 <attribute name="SPICEGROUND" value=""/>
@@
 <part name="U$1" library="untitled" library_urn="urn:adsk.eagle:library:8804918" deviceset="POT-SWITCH" device="" package3d_urn="urn:adsk.eagle:package:8842586/3"/>
 <part name="Q2" library="transistor-power" library_urn="urn:adsk.eagle:library:400" deviceset="PMOSFET_N" device="TO220BV" package3d_urn="urn:adsk.eagle:package:29484/3" value="P16NF06L"/>
+<part name="U$2" library="untitled" library_urn="urn:adsk.eagle:library:8804918" deviceset="VREG-AMS1117-1.5" device="" package3d_urn="urn:adsk.eagle:package:9947855/1"/>
 </parts>
 <sheets>
@@
 </plain>
 <instances>
-<instance part="IC1" gate="A" x="12.7" y="71.12" smashed="yes">
-<attribute name="NAME" x="5.08" y="76.835" size="1.778" layer="95"/>
-<attribute name="VALUE" x="5.08" y="74.295" size="1.778" layer="96"/>
-</instance>
 <instance part="GND1" gate="1" x="-5.08" y="10.16" smashed="yes">
 <attribute name="VALUE" x="-7.62" y="7.62" size="1.778" layer="96"/>
@@
 <attribute name="VALUE" x="111.76" y="40.64" size="1.778" layer="96"/>
 </instance>
+<instance part="U$2" gate="G$1" x="12.7" y="71.12" smashed="yes">
+<attribute name="NAME" x="15.24" y="63.5" size="1.778" layer="95" font="vector"/>
+<attribute name="VALUE" x="15.24" y="60.96" size="1.778" layer="96" font="vector"/>
+</instance>
 </instances>
 <busses>
@@
 <net name="GND" class="0">
 <segment>
-<pinref part="IC1" gate="A" pin="GND"/>
 <wire x1="12.7" y1="63.5" x2="12.7" y2="15.24" width="0.1524" layer="91"/>
 <wire x1="-5.08" y1="15.24" x2="0" y2="15.24" width="0.1524" layer="91"/>
@@
 <junction x="63.5" y="15.24"/>
 <pinref part="U$1" gate="G$1" pin="P$3"/>
+<pinref part="U$2" gate="G$1" pin="GND"/>
 </segment>
 </net>
@@
 <segment>
 <wire x1="25.4" y1="71.12" x2="25.4" y2="45.72" width="0.1524" layer="91"/>
-<pinref part="IC1" gate="A" pin="VO"/>
-<wire x1="25.4" y1="71.12" x2="22.86" y2="71.12" width="0.1524" layer="91"/>
 <wire x1="27.94" y1="71.12" x2="25.4" y2="71.12" width="0.1524" layer="91"/>
 <junction x="25.4" y="71.12"/>
 <pinref part="R1" gate="G$1" pin="1"/>
 <pinref part="C2" gate="G$1" pin="+"/>
+<wire x1="20.32" y1="71.12" x2="22.86" y2="71.12" width="0.1524" layer="91"/>
+<wire x1="22.86" y1="71.12" x2="25.4" y2="71.12" width="0.1524" layer="91"/>
+<wire x1="20.32" y1="68.58" x2="22.86" y2="68.58" width="0.1524" layer="91"/>
+<wire x1="22.86" y1="68.58" x2="22.86" y2="71.12" width="0.1524" layer="91"/>
+<junction x="22.86" y="71.12"/>
+<pinref part="U$2" gate="G$1" pin="OUT"/>
+<pinref part="U$2" gate="G$1" pin="OUT@1"/>
 </segment>
 </net>
 <net name="VCC" class="0">
 <segment>
-<pinref part="IC1" gate="A" pin="VI"/>
-<wire x1="2.54" y1="71.12" x2="0" y2="71.12" width="0.1524" layer="91"/>
 <wire x1="0" y1="71.12" x2="-5.08" y2="71.12" width="0.1524" layer="91"/>
 <wire x1="-5.08" y1="71.12" x2="-5.08" y2="63.5" width="0.1524" layer="91"/>
@@
 <pinref part="U$1" gate="G$2" pin="P$1"/>
 <wire x1="-7.62" y1="63.5" x2="-5.08" y2="63.5" width="0.1524" layer="91"/>
+<wire x1="0" y1="71.12" x2="5.08" y2="71.12" width="0.1524" layer="91"/>
+<pinref part="U$2" gate="G$1" pin="IN"/>
 </segment>
 </net>

Commit message: Minor changes in footprints
Parts:
- removed R6: 0.05, rcl:R-EU_R2512
- added R3: 220, rcl:R-EU_R1206
- R4: value 220 -> 10k
- R5: value 10k -> 0.05; device rcl:R-EU_R1206 -> rcl:R-EU_R2512
- renumbered IC2 to IC1, Q2 to Q1, U$1 to POT1, U$2 to U1, U$3 to J1, U$4 to J2
Connections:
- net GND: now also R5.2; no longer R6.2
- net N$6: now also R3.2; no longer R4.2
- net N$7: now also R3.1; no longer R4.1
- net N$8: now also R4.2; no longer R5.2
- net N$9: now also R4.1; no longer R6.1
Other:
- moved on the sheet: R4, R5
